File: telemetry-rusolar-rework.kicad_pcb (KiCad board)
At the start: 4 copper layers, 109.1 x 84.1 mm, 151 parts, among them IC1 TLV62569DBVR, IC2 TPS2113APW, J1 USART Debug, J10 JP, J11 USB_B_Micro, J12 I2C, J13 GR2, J14 GR1, J15 N_GR1, J16 47219-2001, J2 SPI, J3 MDT420E01001, J4 CAN, J5 Power Out, J6 Power In 12V, J7 SF72S006VBAR2500, J8 SWD, J9 N_GR2, U1 TPS54302, U2 TJA1051TK-3, U3 STM32H725VETx, Y1 50MHz

Commit message: Added changes
Parts:
- removed J15: N_GR1, Connector_PinSocket_2.00mm:PinSocket_1x05_P2.00mm_Vertical
- removed J9: N_GR2, Connector_PinSocket_2.00mm:PinSocket_1x16_P2.00mm_Vertical
- added J17: N_GR1, Connector_PinSocket_2.00mm:PinSocket_1x20_P2.00mm_Vertical, F.Cu at (62.8, 98.2)
- C12: footprint Capacitor_SMD:C_0603_1608Metric_Pad1.08x0.95mm_HandSolder -> Capacitor_SMD:C_0805_2012Metric_Pad1.18x1.45mm_HandSolder
- C47: footprint Capacitor_SMD:C_0805_2012Metric_Pad1.18x1.45mm_HandSolder -> Capacitor_SMD:C_0603_1608Metric_Pad1.08x0.95mm_HandSolder
- J1, J12: footprint Connector_PinSocket_2.00mm:PinSocket_1x02_P2.00mm_Vertical -> Connector_PinHeader_2.00mm:PinHeader_1x02_P2.00mm_Vertical
- J2: footprint Connector_PinSocket_2.00mm:PinSocket_1x03_P2.00mm_Vertical -> Connector_PinHeader_2.00mm:PinHeader_1x03_P2.00mm_Vertical
- R11: value 500 -> 167
- R5: footprint Resistor_SMD:R_0603_1608Metric_Pad0.98x0.95mm_HandSolder -> Resistor_SMD:R_0805_2012Metric_Pad1.20x1.40mm_HandSolder
- moved C12 0.30 mm to (24.5, 163.0)
- moved R5 0.10 mm to (40.6, 143.5)
- moved C47 0.06 mm to (67.2, 139.8)
Routing:
- net GND: track 190.0 -> 179.9 mm, vias 203 -> 208
- net /blue-note-card/RTX: track 55.3 -> 53.3 mm
- net /blue-note-card/CTX: track 53.4 -> 51.5 mm
- net /blue-note-card/AUX3: track 22.3 -> 23.2 mm
- net PE5: track 95.4 -> 96.2 mm
- net PB11: track 101.0 -> 101.8 mm
- net /blue-note-card/VACT_GPS_OUT: track 41.7 -> 42.5 mm
- net /blue-note-card/VACT_GPS_IN: track 39.7 -> 40.5 mm
- net /blue-note-card/SDA: track 29.2 -> 30.0 mm
- net /blue-note-card/AUX_TX: track 13.5 -> 14.3 mm
- net /blue-note-card/AUX_NCHARGING: track 33.6 -> 34.4 mm
- net /blue-note-card/AUX4: track 20.1 -> 20.9 mm
- net /blue-note-card/AUX2: track 24.6 -> 25.4 mm
- net /blue-note-card/AUX1: track 26.8 -> 27.6 mm
- net /blue-note-card/AUX_RX: track 15.5 -> 16.3 mm
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Other:
- board text added: "Fuse"
- board text added: "MISO"
- board text added: "MOSI"
- board text added: "SCK"
- board text removed: "NOT USED"

Commit message: Fixed USB VSENSE, fixed things
Parts:
- removed C62: 100n, Capacitor_SMD:C_0603_1608Metric_Pad1.08x0.95mm_HandSolder
- removed D1: PESD2USB3UV, Package_TO_SOT_SMD:SOT-23W
- removed D8: VESD05A1-02VHG3-08, SamacSys_Parts:VESD05A102VHG308
- removed FB1: FerriteBead, Inductor_SMD:L_0805_2012Metric_Pad1.05x1.20mm_HandSolder
- removed J6: Power In 12V, Connector_PinSocket_2.54mm:PinSocket_1x02_P2.54mm_Vertical
- added C63: 100n, Capacitor_SMD:C_0603_1608Metric_Pad1.08x0.95mm_HandSolder, F.Cu at (82.9, 165.9)
- added D2: ESDA7P60-1U1M, SamacSys_Parts:ESDA7P601U1M, F.Cu at (72.0, 168.0)
- added F2: Fuse, Fuse:Fuse_0603_1608Metric_Pad1.05x0.95mm_HandSolder, F.Cu at (81.2, 171.9)
- added IC3: USBLC6-2P6, SamacSys_Parts:USBLC62P6, F.Cu at (77.1, 170.4)
- added J9: 53048-0210, SamacSys_Parts:SHDRRA2W35P0X125_1X2_425X550X350P, F.Cu at (59.0, 172.5)
- added R36: 33k, Resistor_SMD:R_0603_1608Metric_Pad0.98x0.95mm_HandSolder, F.Cu at (81.2, 170.3)
- added R37: 82k, Resistor_SMD:R_0603_1608Metric_Pad0.98x0.95mm_HandSolder, F.Cu at (83.0, 168.7)
- added R38: 10k, Resistor_SMD:R_0603_1608Metric_Pad0.98x0.95mm_HandSolder, F.Cu at (60.3, 163.9)
- C56: value 100n -> 1u; footprint Capacitor_SMD:C_0603_1608Metric_Pad1.08x0.95mm_HandSolder -> Capacitor_SMD:C_0805_2012Metric_Pad1.18x1.45mm_HandSolder
- C57: value 1u -> 100n; footprint Capacitor_SMD:C_0805_2012Metric_Pad1.18x1.45mm_HandSolder -> Capacitor_SMD:C_0603_1608Metric_Pad1.08x0.95mm_HandSolder
- J4: value CAN -> 53048-0210; footprint Connector_PinSocket_2.00mm:PinSocket_1x02_P2.00mm_Vertical -> SamacSys_Parts:SHDRRA2W35P0X125_1X2_425X550X350P
- R34, R35: value 1k5 -> 470
- moved J4 51.4 mm to (26.0, 133.4)
- moved J17 7.20 mm to (62.8, 91.0)
- moved JP1 7.20 mm to (89.7, 95.4)
- moved H1 7.10 mm to (23.6, 92.5)
- moved H4 7.10 mm to (125.5, 92.4)
- moved C22 3.55 mm to (118.0, 109.7)
- moved C23 3.55 mm to (112.7, 124.4)
- moved C24 3.55 mm to (116.5, 124.4)
- moved C25 3.55 mm to (120.4, 124.4)
- moved C26 3.55 mm to (58.3, 96.7)
- moved C28 3.55 mm to (54.8, 96.7)
- moved C29 3.55 mm to (51.2, 96.7)
- moved C50 3.55 mm to (51.0, 94.7)
- moved C51 3.55 mm to (48.8, 121.6)
- moved C52 3.55 mm to (48.8, 118.2)
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Connections:
- C16 pad 1: +3.3V Buck -> +5V
- C17 pad 1: +3.3V Buck -> +5V
- C56 pad 1: GND -> VBUS
- C56 pad 2: VBUS -> GND
- C57 pad 1: GND -> VBUS
- C57 pad 2: VBUS -> GND
- J11 pad 2: /USB_D- -> Net-(IC3-I/O2_2)
- J11 pad 3: /USB_D+ -> Net-(IC3-I/O1_2)
- J11 pad 6: Net-(J11-Shield) -> unconnected-(J11-Shield-Pad6)
- J13 pad 9: /PA9 -> unconnected-(J13-Pin_9-Pad9)
- J4 pad 1: /CAN_N -> +12V In
- J4 pad 2: /CAN_P -> GND
- R7 pad 1: +3.3V Buck -> +5V
- U2 pad 3: +3.3V Buck -> +5V
- U2 pad 8: unconnected-(U2-S-Pad8) -> Net-(U2-S)
- U3 pad 67: /PA9 -> /VSENSE_USB
Routing:
- net /PA9: track 65.0 -> 0.00 mm, vias 1 -> 0
- net VBUS: track 44.9 -> 77.7 mm
- net +5V: track 47.5 -> 73.4 mm
- net Net-(J11-Shield): track 20.1 -> 0.00 mm
- net /VSENSE_USB: track 0.00 -> 16.6 mm, vias 0 -> 2
- net +3.3V Buck: track 191.3 -> 178.2 mm, vias 38 -> 37
- net GND: track 179.9 -> 191.4 mm, vias 208 -> 197
- net PB10: track 99.2 -> 106.4 mm
- net PE5: track 96.2 -> 103.4 mm
- net PB11: track 101.8 -> 108.6 mm
- net Net-(IC3-I/O1_2): track 0.00 -> 6.72 mm, vias 0 -> 2
- net Net-(IC3-I/O2_2): track 0.00 -> 6.19 mm, vias 0 -> 2
- net /USB_D-: track 16.5 -> 10.9 mm
- net /USB_D+: track 16.5 -> 10.9 mm
- net /blue-note-card/SCL: track 32.2 -> 35.8 mm
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Other:
- board size 109.1 x 84.1 mm -> 109.1 x 91.2 mm
- board text added: "X"
- board text removed: "PA9"
- board text removed: "USB"

Commit message: Fixed things
Parts:
- removed C54, C55, C60, C61: 100n, Capacitor_SMD:C_0603_1608Metric_Pad1.08x0.95mm_HandSolder
- removed D4: 5V_S, LED_SMD:LED_0805_2012Metric_Pad1.15x1.40mm_HandSolder
- removed IC2: TPS2113APW, SamacSys_Parts:NE555DR
- removed J8: SWD, SamacSys_Parts:FTSH-105-XX-YYY-DV-K-A
- removed R10: 36k, Resistor_SMD:R_0805_2012Metric_Pad1.20x1.40mm_HandSolder
- removed R11: 167, Resistor_SMD:R_0603_1608Metric_Pad0.98x0.95mm_HandSolder
- removed R27: 5.1k, Resistor_SMD:R_0603_1608Metric_Pad0.98x0.95mm_HandSolder
- removed R31: 2k2, Resistor_SMD:R_0805_2012Metric_Pad1.20x1.40mm_HandSolder
- removed S4: RKB2SJM250SMTR_LFS, SamacSys_Parts:RKB2SJM250SMTRLFS
- added C62: 100n, Capacitor_SMD:C_0603_1608Metric_Pad1.08x0.95mm_HandSolder, F.Cu at (46.1, 94.6)
- added C64: 10u, Capacitor_SMD:C_0805_2012Metric_Pad1.18x1.45mm_HandSolder, F.Cu at (45.9, 92.7)
- added C65: 1u, Capacitor_SMD:C_0805_2012Metric_Pad1.18x1.45mm_HandSolder, F.Cu at (22.6, 97.2)
- added C66: 100n, Capacitor_SMD:C_0603_1608Metric_Pad1.08x0.95mm_HandSolder, F.Cu at (25.6, 96.0)
- added C69: 100n, Capacitor_SMD:C_0603_1608Metric_Pad1.08x0.95mm_HandSolder, F.Cu at (30.8, 94.0)
- added C70: 1u, Capacitor_SMD:C_0805_2012Metric_Pad1.18x1.45mm_HandSolder, F.Cu at (51.6, 91.6)
- added C71: 100n, Capacitor_SMD:C_0603_1608Metric_Pad1.08x0.95mm_HandSolder, F.Cu at (53.7, 91.3)
- added C74: 1u, Capacitor_SMD:C_0805_2012Metric_Pad1.18x1.45mm_HandSolder, F.Cu at (57.6, 124.0)
- added C75: 100n, Capacitor_SMD:C_0603_1608Metric_Pad1.08x0.95mm_HandSolder, F.Cu at (55.6, 124.1)
- added D1: ESP_PWR, LED_SMD:LED_0805_2012Metric_Pad1.15x1.40mm_HandSolder, F.Cu at (42.8, 93.6)
- added IC4: TPS22917DBVR, SamacSys_Parts:SOT95P280X145-6N, F.Cu at (26.1, 98.8)
- added IC5: TPS22917DBVR, SamacSys_Parts:SOT95P280X145-6N, F.Cu at (57.0, 91.5)
- added IC6: TPS22917DBVR, SamacSys_Parts:SOT95P280X145-6N, F.Cu at (52.5, 124.0)
- added J18: SWD, Connector_PinHeader_2.00mm:PinHeader_1x06_P2.00mm_Vertical, F.Cu at (99.1, 148.7)
- added J19: ESP GPIOs, Connector_PinSocket_2.00mm:PinSocket_1x05_P2.00mm_Vertical, F.Cu at (25.3, 104.6)
- added J6: UART, Connector_PinHeader_2.00mm:PinHeader_1x02_P2.00mm_Vertical, F.Cu at (25.3, 116.6)
- added R39: 100k, Resistor_SMD:R_0805_2012Metric_Pad1.20x1.40mm_HandSolder, F.Cu at (111.3, 133.8)
- added R40: 10k, Resistor_SMD:R_0603_1608Metric_Pad0.98x0.95mm_HandSolder, F.Cu at (30.8, 92.2)
- added R41: 10k, Resistor_SMD:R_0603_1608Metric_Pad0.98x0.95mm_HandSolder, F.Cu at (39.5, 116.8)
- added R42: 100k, Resistor_SMD:R_0805_2012Metric_Pad1.20x1.40mm_HandSolder, F.Cu at (111.3, 129.9)
- added S5: 209-2MS, SamacSys_Parts:2092MS, F.Cu at (106.8, 129.0)
- added S6: ESP_EN_S, SamacSys_Parts:RKB2SJM250SMTRLFS, F.Cu at (36.5, 92.2)
- added S7: ESP_BOOT_S, SamacSys_Parts:RKB2SJM250SMTRLFS, F.Cu at (33.8, 118.7)
- added U4: ESP32-WROOM-32U, RF_Module:ESP32-WROOM-32U, F.Cu at (38.9, 105.9)
- R12: value 10k -> 2k2; footprint Resistor_SMD:R_0805_2012Metric_Pad1.20x1.40mm_HandSolder -> Resistor_SMD:R_0603_1608Metric_Pad0.98x0.95mm_HandSolder
- R26: value 5.1k -> 1k5
- R32, R33, R8: value 1k5 -> 470
- R9: value 157k -> 2k2; footprint Resistor_SMD:R_0805_2012Metric_Pad1.20x1.40mm_HandSolder -> Resistor_SMD:R_0603_1608Metric_Pad0.98x0.95mm_HandSolder
- moved R26 68.6 mm to (42.3, 90.8), turned to 180 degrees
- moved R9 48.6 mm to (84.0, 135.2), turned to 0 degrees
- moved R12 34.6 mm to (44.0, 119.0), turned to 180 degrees
- moved C7 15.5 mm to (47.4, 155.7)
- moved C9 15.5 mm to (47.2, 157.9)
- moved C12 14.5 mm to (36.0, 154.3)
- moved C21 14.5 mm to (39.7, 159.6)
- moved R6 14.5 mm to (39.3, 155.2)
- moved IC1 14.5 mm to (43.4, 154.2)
- moved R14 14.5 mm to (39.4, 152.6)
- moved C15 14.5 mm to (34.9, 159.7)
- moved C20 14.5 mm to (37.3, 159.7)
- moved L1 14.5 mm to (43.1, 157.8)
- moved H5 1.45 mm to (90.5, 109.5)
- moved C53 0.81 mm to (46.8, 117.9)
Connections:
- net /PA1 renamed PA1
- C16 pad 1: +5V -> +5V Buck
- C17 pad 1: +5V -> +5V Buck
- C26 pad 2: +5V -> +5V NOTE
- C28 pad 2: +5V -> +5V NOTE
- C29 pad 2: +5V -> +5V NOTE
- C50 pad 2: +5V -> +5V NOTE
- C51 pad 2: +3.3V Buck -> +3.3V NOTE
- C52 pad 2: +3.3V Buck -> +3.3V NOTE
- C53 pad 2: +3.3V Buck -> +3.3V NOTE
- C7 pad 2: +5V -> +5V Buck
- C9 pad 1: +5V -> +5V Buck
- IC1 pad 1: +5V -> +5V Buck
- IC1 pad 4: +5V -> +5V Buck
- J14 pad 10: /PA0 -> PA0
- J14 pad 18: PB10 -> PB10_PIN_HEADER
- J17 pad 3: PB10 -> PB10_PIN_HEADER
- J3 pad 2: +3.3V Buck -> +3.3V NOTE
- J3 pad 4: +3.3V Buck -> +3.3V NOTE
- J3 pad 62: PB10 -> PB10_PIN_HEADER
- J3 pad 65: /blue-note-card/N_BOOT -> unconnected-(J3-Pad65)
- J3 pad 70: +5V -> +5V NOTE
- J3 pad 72: +5V -> +5V NOTE
- J3 pad 74: +5V -> +5V NOTE
- J5 pad 2: +5V -> +5V Buck
- R12 pad 2: +5V -> PA0
- R26 pad 1: /blue-note-card/N_NRST -> +3.3V ESP
- R26 pad 2: +3.3V Buck -> Net-(D1-A)
- R29 pad 1: +5V -> +5V Buck
- R7 pad 1: +5V -> +5V Buck
- R9 pad 1: +5V Buck -> PB10
- R9 pad 2: Net-(IC2-VSNS) -> PB10_PIN_HEADER
- U2 pad 3: +5V -> +5V Buck
- U3 pad 25: /PA0 -> PA0
Routing:
- net /ESP32-Wifi/ESP_ON: track 0.00 -> 117.8 mm, vias 0 -> 2
- net /ESP32-Wifi/NOTE_ON: track 0.00 -> 100.8 mm, vias 0 -> 2
- net PB10: track 106.4 -> 27.9 mm
- net PB10_PIN_HEADER: track 0.00 -> 78.5 mm, vias 0 -> 1
- net +5V: track 73.4 -> 0.00 mm, vias 20 -> 0
- net PA0: track 0.00 -> 70.9 mm, vias 0 -> 2
- net /blue-note-card/N_BOOT: track 69.7 -> 0.00 mm, vias 2 -> 0
- net PA1: track 18.5 -> 69.8 mm, vias 1 -> 3
- net +3.3V Buck: track 178.2 -> 223.5 mm, vias 37 -> 35
- net VBUS: track 77.7 -> 40.8 mm
- net +3.3V ESP: track 0.00 -> 33.9 mm, vias 0 -> 2
- net /NRST: track 54.1 -> 85.8 mm, vias 4 -> 3
- net /SWO: track 19.7 -> 44.3 mm
- net GND: track 191.4 -> 214.9 mm, vias 197 -> 202
- net /SWD_CLK: track 14.5 -> 37.4 mm
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- added copper zone on F.Cu, net +3.3V NOTE
- added copper zone on In2.Cu, net +5V Buck
- added copper zone on F.Cu, net +5V NOTE
- removed copper zone on F.Cu, net +5V
- removed copper zone on In2.Cu, net +5V
Other:
- board text added: "3.3"
- board text added: "BOOT"
- board text added: "CLK"
- board text added: "EPWR"
- board text added: "ESP BOOT"
- board text added: "ESP ON"
- board text added: "ESP UART"
- board text added: "E_NRST"
- board text added: "GPIOs"
- board text added: "IO"
- board text added: "IO12"
- board text added: "IO13"
- board text added: "IO2"
- board text added: "IO4"
- board text added: "IO5"
- board text added: "NOTE NRST"
- board text added: "NOTE ON"
- board text added: "PA0*"
- board text added: "PA0* (UART4) -> RXD0 ESP"
- board text added: "PA1*"
- board text added: "PA1* (UART4) -> TXD0 ESP"
- board text added: "PA4* -> CAN_ERR LED"
- board text added: "PB1* -> CAN TX LED"
- board text added: "PB2* -> CAN RX LED"
- board text added: "PB5* -> USR2 LED"
- board text added: "PE2* -> USR1 LED"
- board text added: "PE5* -> [Note] ATTN"
- board text added: "QUANG - STM32H725VE - BlueNoteCard - ESP32-WROOM-32U"
- board text added: "SWO"
- board text added: "USR1"
- board text added: "USR2"
- board text removed: "5V STAT"
- board text removed: "BOOT0"
- board text removed: "N_BOOT"
- board text removed: "N_NRST"
- board text removed: "PA0"
- board text removed: "PA1"
- board text removed: "PA4* -> CAN_ERR"
- board text removed: "PB1* -> TX"
- board text removed: "PB2* -> RX"
- board text removed: "PB5* -> USER LED 2"
- board text removed: "PE2* -> USER LED 1"
- board text removed: "PE5* -> ATTN"
- board text removed: "Quang Dinh Bui."
- board text removed: "Rev 1.1.1 4/12/2025"
- board text removed: "USER LED 1"
- board text removed: "USER LED 2"
- board text removed: "VBUS"

Commit message: Fixed a lot of things
Parts:
- removed R12: 2k2, Resistor_SMD:R_0603_1608Metric_Pad0.98x0.95mm_HandSolder
- added R10: 2k2, Resistor_SMD:R_0603_1608Metric_Pad0.98x0.95mm_HandSolder, F.Cu at (44.8, 117.9)
- moved Y1 0.48 mm to (73.1, 135.2)
Connections:
- J11 pad 6: unconnected-(J11-Shield-Pad6) -> GND
- J6 pad 1: PA1 -> /ESP32-Wifi/ESP_UART0_TX
- J6 pad 2: PA0 -> /ESP32-Wifi/ESP_UART0_RX
- U4 pad 27: unconnected-(U4-IO16-Pad27) -> Net-(U4-IO16)
- U4 pad 28: unconnected-(U4-IO17-Pad28) -> PA1
- U4 pad 34: Net-(U4-RXD0/IO3) -> /ESP32-Wifi/ESP_UART0_RX
- U4 pad 35: PA1 -> /ESP32-Wifi/ESP_UART0_TX
Routing:
- net PA0: track 70.9 -> 47.5 mm
- net /ESP32-Wifi/ESP_UART0_TX: track 0.00 -> 21.2 mm, vias 0 -> 1
- net /ESP32-Wifi/ESP_UART0_RX: track 0.00 -> 20.8 mm, vias 0 -> 1
- net Net-(U4-IO16): track 0.00 -> 17.6 mm, vias 0 -> 2
- net PA1: track 69.8 -> 62.8 mm
- net Net-(U4-RXD0/IO3): track 5.99 -> 0.00 mm
- net +3.3V Buck: track 223.5 -> 218.3 mm, vias 35 -> 41
- net /PC1: track 23.9 -> 27.7 mm
- net /PC15: track 17.2 -> 19.8 mm
- net /PC2_C: track 17.6 -> 20.2 mm
- net +12V: track 10.1 -> 7.50 mm, vias 11 -> 16
- net /PC0: track 24.3 -> 26.8 mm
- net +5V Buck: track 33.2 -> 30.9 mm, vias 16 -> 21
- net GND: track 214.9 -> 216.7 mm, vias 202 -> 212
- net /PC14: track 17.5 -> 18.8 mm
- added copper zone on In2.Cu, net GND
Other:
- board text added: "ESP UART0"
- board text added: "PA0* (UART4 TX) -> UART2 RX ESP"
- board text added: "PA1* (UART4 RX) -> UART2 TX ESP"
- board text added: "[ALERT] DO NOT SET PA1 as GPIO OUTPUT"
- board text added: "[ALERT] DO NOT SET PB11 as GPIO OUTPUT"
- board text removed: "ESP UART"
- board text removed: "PA0* (UART4) -> RXD0 ESP"
- board text removed: "PA1* (UART4) -> TXD0 ESP"

Commit message: Added temp
Parts:
- R20, R22, R23: value 47k -> 100k
- R21: value 47k -> 90k
Routing:
- net +5V Buck: track 30.9 -> 48.8 mm
- net GND: track 216.7 -> 216.3 mm, vias 212 -> 213
Other:
- board text added: "v1.2.0"
Changed lines of the file:
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@@
 			)
 		)
-		(property "Value" "47k"
+		(property "Value" "100k"
 			(at 0 1.65 90)
 			(layer "F.Fab")
@@
 			)
 		)
-		(property "Value" "47k"
+		(property "Value" "100k"
 			(at 0 1.65 90)
 			(layer "F.Fab")
@@
 			)
 		)
-		(property "Value" "47k"
+		(property "Value" "90k"
 			(at 0 1.65 90)
 			(layer "F.Fab")
@@
 			)
 		)
-		(property "Value" "47k"
+		(property "Value" "100k"
 			(at 0 1.65 90)
 			(layer "F.Fab")
@@
 		(layer "F.SilkS")
 	)
-	(gr_line
-		(start 60.25 92.55)
-		(end 62 92.55)
-		(stroke
-			(width 0.1)
-			(type default)
-		)
-		(layer "F.SilkS")
-	)
 	(gr_poly
 		(pts
@@
 		)
 	)
+	(gr_text "v1.2.0"
+		(at 127 107.9 90)
+		(layer "F.SilkS")
+		(effects
+			(font
+				(size 1 1)
+				(thickness 0.15)
+			)
+			(justify left bottom)
+		)
+	)
 	(gr_text "PD3"
 		(at 115.45 139 0)
@@
 	)
 	(segment
-		(start 65.8875 161.6875)
-		(end 66.3 162.1)
-		(width 0.3)
-		(layer "F.Cu")
-		(net 1)
-	)
-	(segment
 		(start 108.42 167.12)
 		(end 108.4 167.1)
@@
 	)
 	(segment
+		(start 64.7 161.6875)
+		(end 64.7 162.75)
+		(width 0.3)
+		(layer "F.Cu")
+		(net 1)
+	)
+	(segment
 		(start 53.6 143.9)
 		(end 53.6 144.2)
@@
 	)
 	(segment
-		(start 64.7 161.6875)
-		(end 65.8875 161.6875)
-		(width 0.3)
-		(layer "F.Cu")
-		(net 1)
-	)
-	(segment
 		(start 51.45 104.801)
 		(end 52.85 104.801)
@@
 	)
 	(segment
+		(start 64.7 162.75)
+		(end 62.9 164.55)
+		(width 0.3)
+		(layer "F.Cu")
+		(net 1)
+	)
+	(segment
 		(start 70.425 142.4)
 		(end 70.425 140.6875)
@@
 	)
 	(segment
-		(start 47.165 96.95)
-		(end 47.165 94.765)
-		(width 0.3)
-		(layer "F.Cu")
-		(net 1)
-	)
-	(segment
 		(start 28.0375 142.2)
 		(end 27.6 142.2)
@@
 	)
 	(via
-		(at 66.3 162.1)
-		(size 0.7)
-		(drill 0.3)
-		(layers "F.Cu" "B.Cu")
-		(net 1)
-	)
-	(via
 		(at 33.4 135.7)
 		(size 0.7)
@@
 	)
 	(via
+		(at 53.6 93.5)
+		(size 0.7)
+		(drill 0.3)
+		(layers "F.Cu" "B.Cu")
+		(free yes)
+		(net 1)
+	)
+	(via
 		(at 111.9 176.3)
 		(size 0.7)
@@
 	)
 	(via
+		(at 54.4 93.5)
+		(size 0.7)
+		(drill 0.3)
+		(layers "F.Cu" "B.Cu")
+		(free yes)
+		(net 1)
+	)
+	(via
 		(at 113.45 111.501)
 		(size 0.7)
@@
 	)
 	(segment
-		(start 59.05 154.15)
-		(end 57.9125 153.0125)
-		(width 0.3)
+		(start 67 160.6)
+		(end 67 162.6)
+		(width 0.5)
 		(layer "F.Cu")
 		(net 140)
 	)
 	(segment
-		(start 60.45 156.458636)
-		(end 60.45 155.55)
+		(start 42.4375 154.8)
+		(end 42.4375 155.4)
 		(width 0.3)
 		(layer "F.Cu")
@@
 	)
 	(segment
-		(start 42.4375 154.8)
-		(end 42.4375 155.4)
-		(width 0.3)
+		(start 64.7 159.6125)
+		(end 66.0125 159.6125)
+		(width 0.5)
 		(layer "F.Cu")
 		(net 140)
@@
 	)
 	(segment
+		(start 59.7125 153.0125)
+		(end 55.8 153.0125)
+		(width 0.2)
+		(layer "F.Cu")
+		(net 140)
+	)
+	(segment
+		(start 64.7 159.5)
+		(end 64.7 159.6125)
+		(width 0.3)
+		(layer "F.Cu")
+		(net 140)
+	)
+	(segment
+		(start 63.8 165.8)
+		(end 51.4 165.8)
+		(width 0.5)
+		(layer "F.Cu")
+		(net 140)
+	)
+	(segment
+		(start 51.4 165.8)
+		(end 50.8 165.8)
+		(width 0.5)
+		(layer "F.Cu")
+		(net 140)
+	)
+	(segment
+		(start 64.7 159.6125)
+		(end 63.5875 158.5)
+		(width 0.2)
+		(layer "F.Cu")
+		(net 140)
+	)
+	(segment
+		(start 60.8 156.7)
+		(end 60.8 154.1)
+		(width 0.2)
+		(layer "F.Cu")
+		(net 140)
+	)
+	(segment
+		(start 50.8 165.8)
+		(end 48 163)
+		(width 0.5)
+		(layer "F.Cu")
+		(net 140)
+	)
+	(segment
 		(start 33.5125 142.2)
 		(end 33.5125 142.553979)
@@
 	)
 	(segment
-		(start 57.9125 153.0125)
-		(end 55.8 153.0125)
+		(start 64.7 159.6125)
+		(end 64.9125 159.6125)
 		(width 0.3)
 		(layer "F.Cu")
@@
 	)
 	(segment
-		(start 64.7 159.6125)
-		(end 64.9125 159.6125)
-		(width 0.3)
+		(start 62.6 158.5)
+		(end 60.8 156.7)
+		(width 0.2)
 		(layer "F.Cu")
 		(net 140)
 	)
 	(segment
-		(start 59.4 154.5)
-		(end 59.05 154.15)
-		(width 0.3)
+		(start 66.0125 159.6125)
+		(end 67 160.6)
+		(width 0.5)
 		(layer "F.Cu")
 		(net 140)
 	)
 	(segment
-		(start 59.4 154.5)
-		(end 59 154.1)
-		(width 0.3)
+		(start 63.5875 158.5)
+		(end 62.6 158.5)
+		(width 0.2)
 		(layer "F.Cu")
 		(net 140)
@@
 	)
 	(segment
-		(start 62.5625 159.6375)
-		(end 62.5625 158.571136)
-		(width 0.3)
+		(start 60.8 154.1)
+		(end 59.7125 153.0125)
+		(width 0.2)
 		(layer "F.Cu")
 		(net 140)
@@
 	)
 	(segment
-		(start 62.5625 158.571136)
-		(end 60.45 156.458636)
-		(width 0.3)
-		(layer "F.Cu")
-		(net 140)
-	)
-	(segment
-		(start 59 154.1)
-		(end 48.7 154.1)
-		(width 0.3)
+		(start 67 162.6)
+		(end 63.8 165.8)
+		(width 0.5)
 		(layer "F.Cu")
 		(net 140)
@@
 	)
 	(segment
-		(start 60.45 155.55)
-		(end 59.4 154.5)
-		(width 0.3)
-		(layer "F.Cu")
-		(net 140)
-	)
-	(segment
 		(start 61.725 159.6375)
 		(end 62.5625 159.6375)
@@
 	)
 	(via
-		(at 48.7 154.1)
+		(at 48 163)
 		(size 0.7)
 		(drill 0.3)
@@
 	)
 	(segment
-		(start 53.6 93.5)
-		(end 55.8 93.5)
+		(start 49.2 97.9)
+		(end 52.5 94.6)
 		(width 0.2)
 		(layer "B.Cu")
@@
 	)
 	(segment
-		(start 53.7 122)
-		(end 50.7 122)
+		(start 49.2 120.5)
+		(end 49.2 97.9)
 		(width 0.2)
 		(layer "B.Cu")
@@
 	)
 	(segment
-		(start 49.2 120.5)
-		(end 49.2 97.9)
+		(start 54.7 94.6)
+		(end 55.8 93.5)
 		(width 0.2)
 		(layer "B.Cu")
@@
 	)
 	(segment
-		(start 49.2 97.9)
-		(end 53.6 93.5)
+		(start 53.7 122)
+		(end 50.7 122)
+		(width 0.2)
+		(layer "B.Cu")
+		(net 168)
+	)
+	(segment
+		(start 52.5 94.6)
+		(end 54.7 94.6)
 		(width 0.2)
 		(layer "B.Cu")
@@
 				(xy 51.1 97.4) (xy 49.6 97.4) (xy 49.6 95.7) (xy 46.3 95.7) (xy 46.3 93.8) (xy 46 93.8) (xy 46 91.9)
 				(xy 52.8 91.9) (xy 52.8 91.5) (xy 54.6 91.5) (xy 54.6 91) (xy 56.5 91) (xy 56.5 91.9) (xy 54.8 91.9)
-				(xy 54.8 93.5) (xy 51.1 93.5)
+				(xy 54.8 94) (xy 53 94) (xy 53 93.5) (xy 51.1 93.5)
 			)
 		)
